File: current_sensor.kicad_pcb (KiCad board)
At the start: 2 copper layers, 32 x 23 mm, 16 parts, among them P1 CONN_01X02, P2 CONN_01X03, P3 CONN_01X01, P4 CONN_01X01, U1 ACS712, U2 OPA344

Commit message: Added changed files
Parts:
- added D1: LED, EE:LED-0603_NEW, F.Cu at (140.2, 54.4)
- added R3: 1K, Resistors_SMD:R_0603_HandSoldering, F.Cu at (139.2, 57.4)
- U2: value OPA344 -> LM_321
- moved LOGO 0.13 mm to (138.7, 44.5)
Connections:
- U2 pad 1: Net-(C5-Pad1) -> Net-(C3-Pad2)
- U2 pad 3: Net-(C3-Pad2) -> Net-(C5-Pad2)
- U2 pad 4: Net-(C5-Pad2) -> Net-(C5-Pad1)
Routing:
- net VCC: track 47.4 -> 62.7 mm, vias 0 -> 1
- net Net-(C3-Pad2): track 16.9 -> 22.6 mm, vias 0 -> 1
- net Net-(C5-Pad2): track 25.5 -> 20.6 mm
- net Net-(C5-Pad1): track 17.8 -> 21.1 mm, vias 1 -> 2
- net GND: track 76.6 -> 79.2 mm
- net Net-(D1-Pad1): track 0.00 -> 2.33 mm
