File: current_sensor.sch (KiCad schematic (older format))
At the start: 15 parts, among them P1 CONN_01X02, P2 CONN_01X03, P3 CONN_01X01, P4 CONN_01X01, U1 ACS712, U2 OPA344

Commit message: Added changed files
Parts:
- removed U2: OPA344, symbol OPA344
- added D1: LED, symbol LED
- added R3: 1K, symbol R
- added U2: LM_321, symbol LM_321
Connections:
- net GND: now also D1.2 (K), U2.2 (V-)
- net VCC: now also R3.2, U2.5 (V+)
- net at C5.1, P2.2 (P2), R2.1: now also U2.4 (OUT)
- net at C3.2, RV1.2: now also U2.1 (IN+)
- net at C5.2, R2.2, RV2.2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: now also U2.3 (IN-)
- new net: D1.1 (A), R3.1
Other:
- moved on the sheet: C4
Changed lines of the file:
@@
-$EndComp
-$Comp
-L OPA344 U2
-U 1 1 560A3575
-P 6250 2200
-F 0 "U2" H 6400 1700 60  0000 C CNN
-F 1 "OPA344" H 6400 1800 60  0000 C CNN
-F 2 "" H 6250 2200 60  0000 C CNN
-F 3 "" H 6250 2200 60  0000 C CNN
-	1    6250 2200
-	1    0    0    -1
 $EndComp
 $Comp
@@
 L GND #PWR06
 U 1 1 560A3927
-P 6450 2800
-F 0 "#PWR06" H 6450 2550 60  0001 C CNN
-F 1 "GND" H 6450 2650 60  0000 C CNN
-F 2 "" H 6450 2800 60  0000 C CNN
-F 3 "" H 6450 2800 60  0000 C CNN
-	1    6450 2800
+P 6500 2800
+F 0 "#PWR06" H 6500 2550 60  0001 C CNN
+F 1 "GND" H 6500 2650 60  0000 C CNN
+F 2 "" H 6500 2800 60  0000 C CNN
+F 3 "" H 6500 2800 60  0000 C CNN
+	1    6500 2800
 	1    0    0    -1
 $EndComp
@@
 L VCC #PWR07
 U 1 1 560A3985
-P 6450 1600
-F 0 "#PWR07" H 6450 1450 60  0001 C CNN
-F 1 "VCC" H 6450 1750 60  0000 C CNN
-F 2 "" H 6450 1600 60  0000 C CNN
-F 3 "" H 6450 1600 60  0000 C CNN
-	1    6450 1600
+P 6500 1600
+F 0 "#PWR07" H 6500 1450 60  0001 C CNN
+F 1 "VCC" H 6500 1750 60  0000 C CNN
+F 2 "" H 6500 1600 60  0000 C CNN
+F 3 "" H 6500 1600 60  0000 C CNN
+	1    6500 1600
 	1    0    0    -1
 $EndComp
@@
 L C C4
 U 1 1 560A39E4
-P 6700 1650
-F 0 "C4" H 6750 1750 50  0000 L CNN
-F 1 "0.1uF" H 6750 1550 50  0000 L CNN
-F 2 "" H 6738 1500 30  0000 C CNN
-F 3 "" H 6700 1650 60  0000 C CNN
-	1    6700 1650
+P 6800 1650
+F 0 "C4" H 6850 1750 50  0000 L CNN
+F 1 "0.1uF" H 6850 1550 50  0000 L CNN
+F 2 "" H 6838 1500 30  0000 C CNN
+F 3 "" H 6800 1650 60  0000 C CNN
+	1    6800 1650
 	0    1    1    0
 $EndComp
@@
 L GND #PWR08
 U 1 1 560A3AFA
-P 6950 1800
-F 0 "#PWR08" H 6950 1550 60  0001 C CNN
-F 1 "GND" H 6950 1650 60  0000 C CNN
-F 2 "" H 6950 1800 60  0000 C CNN
-F 3 "" H 6950 1800 60  0000 C CNN
-	1    6950 1800
+P 7050 1800
+F 0 "#PWR08" H 7050 1550 60  0001 C CNN
+F 1 "GND" H 7050 1650 60  0000 C CNN
+F 2 "" H 7050 1800 60  0000 C CNN
+F 3 "" H 7050 1800 60  0000 C CNN
+	1    7050 1800
 	1    0    0    -1
 $EndComp
@@
 	5600 2500 5600 2550
 Wire Wire Line
-	6450 2500 6450 2800
-Wire Wire Line
-	6450 1900 6450 1600
-Wire Wire Line
-	6500 1650 6450 1650
-Connection ~ 6450 1650
-Wire Wire Line
-	6900 1650 6950 1650
-Wire Wire Line
-	6950 1650 6950 1800
-Wire Wire Line
 	6050 850  6050 2100
 Wire Wire Line
@@
 NoConn ~ 5050 850
 NoConn ~ 5050 1400
+$Comp
+L LM_321 U2
+U 1 1 562F5388
+P 6250 2200
+F 0 "U2" H 6350 1700 60  0000 C CNN
+F 1 "LM_321" H 6400 1800 60  0000 C CNN
+F 2 "" H 6250 2200 60  0000 C CNN
+F 3 "" H 6250 2200 60  0000 C CNN
+	1    6250 2200
+	1    0    0    -1
+$EndComp
+Wire Wire Line
+	6500 2450 6500 2800
+Wire Wire Line
+	6500 1600 6500 1950
+Wire Wire Line
+	6500 1650 6600 1650
+Wire Wire Line
+	7050 1800 7050 1650
+Wire Wire Line
+	7050 1650 7000 1650
+Connection ~ 6500 1650
+$Comp
+L R R3
+U 1 1 562F597B
+P 2500 1800
+F 0 "R3" V 2580 1800 50  0000 C CNN
+F 1 "1K" V 2507 1801 50  0000 C CNN
+F 2 "" V 2430 1800 30  0000 C CNN
+F 3 "" H 2500 1800 30  0000 C CNN
+	1    2500 1800
+	-1   0    0    1
+$EndComp
+$Comp
+L LED D1
+U 1 1 562F5B13
+P 2500 2350
+F 0 "D1" H 2500 2450 50  0000 C CNN
+F 1 "LED" H 2500 2250 50  0000 C CNN
+F 2 "" H 2500 2350 60  0000 C CNN
+F 3 "" H 2500 2350 60  0000 C CNN
+	1    2500 2350
+	0    1    1    0
+$EndComp
+Wire Wire Line
+	2500 2050 2500 2150
+$Comp
+L GND #PWR011
+U 1 1 562F5C61
+P 2500 2650
+F 0 "#PWR011" H 2500 2400 60  0001 C CNN
+F 1 "GND" H 2500 2500 60  0000 C CNN
+F 2 "" H 2500 2650 60  0000 C CNN
+F 3 "" H 2500 2650 60  0000 C CNN
+	1    2500 2650
+	1    0    0    -1
+$EndComp
+Wire Wire Line
+	2500 2550 2500 2650
+$Comp
+L VCC #PWR012
+U 1 1 562F5D5C
+P 2500 1500
+F 0 "#PWR012" H 2500 1350 60  0001 C CNN
+F 1 "VCC" H 2500 1650 60  0000 C CNN
+F 2 "" H 2500 1500 60  0000 C CNN
+F 3 "" H 2500 1500 60  0000 C CNN
+	1    2500 1500
+	1    0    0    -1
+$EndComp
+Wire Wire Line
+	2500 1500 2500 1550
 $EndSCHEMATC
